File: can_module/can_mcp2515.sch (KiCad schematic (older format))
At the start: 14 parts, among them J201 RJ45, J202 Screw_Terminal_01x02, U201 PESD5V0L2UU_esd_diode, U202 MCP2551-I-SN, U203 MCP2515-xST, Y201 Crystal

Commit message: controller v2 voor testvaart 1 mei
Parts:
- removed J201: RJ45, Connector_RJ:RJ45_Amphenol_54602-x08_Horizontal, symbol Connector:RJ45
- removed J202: Screw_Terminal_01x02, Connector_Phoenix_MC_HighVoltage:PhoenixContact_MCV_1,5_2-G-5.08_1x02_P5.08mm_Vertical, symbol Connector:Screw_Terminal_01x02
- added J201: can, Connector_Phoenix_MC_HighVoltage:PhoenixContact_MCV_1,5_4-G-5.08_1x04_P5.08mm_Vertical, symbol Connector:Screw_Terminal_01x04
- U201: symbol nucleo_can-rescue:PESD5V0L2UU_esd_diode -> zonneboot_parts:PESD5V0L2UU_esd_diode
Connections:
- net can_h: now also J201.1 (Pin_1), J201.3 (Pin_3)
- net can_l: now also J201.2 (Pin_2), J201.4 (Pin_4)
Changed lines of the file:
@@
 	-1   0    0    -1
 $EndComp
-$Comp
-L Connector:RJ45 J201
-U 1 1 6074BA6F
-P 2450 3125
-F 0 "J201" H 2507 3792 50  0000 C CNN
-F 1 "RJ45" H 2507 3701 50  0000 C CNN
-F 2 "Connector_RJ:RJ45_Amphenol_54602-x08_Horizontal" V 2450 3150 50  0001 C CNN
-F 3 "~" V 2450 3150 50  0001 C CNN
-	1    2450 3125
-	0    -1   -1   0
-$EndComp
-Wire Wire Line
-	2150 2725 2150 2675
-Wire Wire Line
-	2050 2675 2050 2725
 Wire Wire Line
 	1450 1775 1450 1475
@@
 $EndComp
 $Comp
-L nucleo_can-rescue:PESD5V0L2UU_esd_diode U201
+L zonneboot_parts:PESD5V0L2UU_esd_diode U201
 U 1 1 6074BA81
 P 1750 1875
+AR Path="/6074BA81" Ref="U201"  Part="1"
+AR Path="/6074414E/6074BA81" Ref="U201"  Part="1"
 F 0 "U201" V 1746 1897 50  0000 R CNN
 F 1 "PESD5V0L2UU_esd_diode" V 1550 2525 50  0000 R CNN
@@
 	1    0    0    -1
 $EndComp
-$Comp
-L Connector:Screw_Terminal_01x02 J202
-U 1 1 6074BB1B
-P 3100 3375
-F 0 "J202" V 2972 3455 50  0000 L CNN
-F 1 "Screw_Terminal_01x02" V 3063 3455 50  0000 L CNN
-F 2 "Connector_Phoenix_MC_HighVoltage:PhoenixContact_MCV_1,5_2-G-5.08_1x02_P5.08mm_Vertical" H 3100 3375 50  0001 C CNN
-F 3 "~" H 3100 3375 50  0001 C CNN
-	1    3100 3375
-	0    1    1    0
-$EndComp
-Text Label 3100 3175 1    50   ~ 0
-can_h
-Text Label 3000 3175 1    50   ~ 0
-can_l
-Text Label 2150 2675 1    50   ~ 0
-can_h
-Text Label 2050 2675 1    50   ~ 0
+Text Label 2600 3000 1    50   ~ 0
+can_h
+Text Label 2500 3000 1    50   ~ 0
+can_l
+Text Label 2400 3000 1    50   ~ 0
+can_h
+Text Label 2300 3000 1    50   ~ 0
 can_l
 Text Label 1400 1475 2    50   ~ 0
@@
 Wire Wire Line
 	1525 1475 1800 1475
+$Comp
+L Connector:Screw_Terminal_01x04 J201
+U 1 1 6076236F
+P 2500 3200
+F 0 "J201" V 2372 3380 50  0000 L CNN
+F 1 "can" V 2463 3380 50  0000 L CNN
+F 2 "Connector_Phoenix_MC_HighVoltage:PhoenixContact_MCV_1,5_4-G-5.08_1x04_P5.08mm_Vertical" H 2500 3200 50  0001 C CNN
+F 3 "~" H 2500 3200 50  0001 C CNN
+	1    2500 3200
+	0    1    1    0
+$EndComp
 $EndSCHEMATC
