File: foil_controller/foil_controller.sch (KiCad schematic (older format))
At the start: 18 parts, among them J1 programming_header, J2 pwr_in, J3 ultra sensor 1, J4 ultra sensor 1, SW1 SW_Push, SW2 SW_Push, SW3 SW_Push, SW4 SW_Push, U1 RS485_module, U2 L7805

Commit message: controller v2 voor testvaart 1 mei
Parts:
- removed R1, R2, R3, R4: 10K, Resistor_THT:R_Axial_DIN0207_L6.3mm_D2.5mm_P7.62mm_Horizontal, symbol Device:R
- removed U1: RS485_module, stroom_shield:RS485_module, symbol stroom_shield:RS485_module
- added C101, C102, C103, C104: 47nf, Capacitor_SMD:C_0603_1608Metric_Pad1.05x0.95mm_HandSolder, symbol Device:C
- added R101, R102, R103, R104: 10K, Resistor_SMD:R_0603_1608Metric_Pad1.05x0.95mm_HandSolder, symbol Device:R
- added SW101: SW_DIP_x02, Button_Switch_THT:SW_DIP_SPSTx02_Slide_6.7x6.64mm_W7.62mm_P2.54mm_LowProfile, symbol Switch:SW_DIP_x02
- added SW102: Encoder_1, Rotary_Encoder:RotaryEncoder_Alps_EC11E-Switch_Vertical_H20mm_CircularMountingHoles, symbol Device:Rotary_Encoder_Switch
- added SW103: Encoder_2, Rotary_Encoder:RotaryEncoder_Alps_EC11E-Switch_Vertical_H20mm_CircularMountingHoles, symbol Device:Rotary_Encoder_Switch
- DS1: footprint Display:WC1602A -> zonneboot_parts:WINSTAR-WH1604A
- J3, J4: footprint Connector:FanPinHeader_1x04_P2.54mm_Vertical -> Connector_Molex:Molex_SL_171971-0004_1x04_P2.54mm_Vertical
Connections:
- net +3V3: now also R101.2, R102.2, R103.2, R104.2
- net +5V: no longer SW1.1, SW2.1, SW3.1, SW4.1
- net GND: now also SW1.1, SW2.1, SW3.1, SW4.1, C101.2, C102.2, C103.2, C104.2, SW102.C, SW102.S1, SW103.C, SW103.S1
- net btn_1: now also BP1.12 (PB4); no longer BP1.17 (PB9)
- net btn_2: now also BP1.13 (PB5); no longer BP1.16 (PB8)
- net btn_3: now also BP1.14 (PB6); no longer BP1.15 (PB7)
- net btn_4: now also BP1.15 (PB7); no longer BP1.14 (PB6)
- net echo_1: now also BP1.10 (PA15); no longer BP1.13 (PB5)
- net echo_2: now also BP1.8 (PA11); no longer BP1.11 (PB3)
- net prog_RX: now also SW101.1
- net prog_TX: now also SW101.2
- net trig_1: now also BP1.11 (PB3); no longer BP1.12 (PB4)
- net trig_2: now also BP1.9 (PA12); no longer BP1.10 (PA15)
- net Encoder2_btn: now reaches BP1.2 (PB13)
- net Encoder2_btn: now also SW103.S2
- net at DS1.11 (D4): no longer BP1.29 (PA4)
- net Encoder2_B: now reaches BP1.3 (PB14)
- net Encoder2_B: now also C103.1, R103.1, SW103.B
- net at DS1.12 (D5): no longer BP1.30 (PA5)
- net at DS1.13 (D6): no longer BP1.31 (PA6)
- net at DS1.14 (D7): no longer BP1.32 (PA7)
- net sheet60828324/can_spi_cs: now reaches BP1.33 (PB0)
- net Encoder2_A: now reaches BP1.4 (PB15)
- net Encoder2_A: now also C104.1, R104.1, SW103.A
- net Encoder1_btn: now reaches BP1.5 (PA8)
- net Encoder1_btn: now also SW102.S2
- new net Encoder1_A: BP1.17 (PB9), C102.1, R102.1, SW102.A
- new net Encoder1_B: BP1.16 (PB8), C101.1, R101.1, SW102.B
- new net Sheet60804332/can_spi_clk: BP1.30 (PA5)
- new net Sheet60804332/can_spi_cs: BP1.29 (PA4)
- new net Sheet60804332/can_spi_miso: BP1.31 (PA6)
- new net Sheet60804332/can_spi_mosi: BP1.32 (PA7)
- new net Sheet6080570A/RX_FROM_USB: SW101.3
- new net Sheet6080570A/TX_FROM_USB: SW101.4
- no-connect marks 0 -> 13
Other:
- moved on the sheet: J2, J3, J4, SW1, SW2, SW3, SW4, U2
