File: foil_io_shield/foil_io_shield.kicad_pcb (KiCad board)
At the start: 2 copper layers, 70.5 x 61.1 mm, 15 parts, among them J1 12v, J2 encoder_header_1, J3 encoder_header_1, U1 LM7805_TO220, U2 NUCLEO-F446RE, U3 RS485_module

Commit message: controller v2 voor testvaart 1 mei
Parts:
- removed ?: , text:label
- removed U3: RS485_module, stroom_shield:RS485_module
- added C201: 100nf, Capacitor_SMD:C_0603_1608Metric_Pad1.05x0.95mm_HandSolder, F.Cu at (185.4, 69.6)
- added C202: 100nf, Capacitor_SMD:C_0603_1608Metric_Pad1.05x0.95mm_HandSolder, F.Cu at (206.2, 76.1)
- added C203: 2pf, Capacitor_SMD:C_0603_1608Metric_Pad1.05x0.95mm_HandSolder, F.Cu at (211.3, 70.4)
- added C204: 2pf, Capacitor_SMD:C_0603_1608Metric_Pad1.05x0.95mm_HandSolder, F.Cu at (211.3, 66.9)
- added J201: can, Connector_Phoenix_MC_HighVoltage:PhoenixContact_MCV_1,5_4-G-5.08_1x04_P5.08mm_Vertical, F.Cu at (207.6, 59.6)
- added JP201: termination, Jumper:SolderJumper-2_P1.3mm_Open_TrianglePad1.0x1.5mm, F.Cu at (186.6, 58.6)
- added R201: 120R, Resistor_SMD:R_0603_1608Metric_Pad1.05x0.95mm_HandSolder, F.Cu at (186.6, 62.5)
- added R202: 47K, Resistor_SMD:R_0603_1608Metric_Pad1.05x0.95mm_HandSolder, F.Cu at (196.0, 72.2)
- added R203: 10K, Resistor_SMD:R_0603_1608Metric_Pad1.05x0.95mm_HandSolder, F.Cu at (203.1, 74.0)
- added U201: PESD5V0L2UU_esd_diode, Package_TO_SOT_SMD:SOT-323_SC-70_Handsoldering, F.Cu at (195.8, 68.6)
- added U202: MCP2551-I-SN, Package_SO:SOIC-8_3.9x4.9mm_P1.27mm, F.Cu at (190.0, 69.7)
- added U203: MCP2515-xST, Package_SO:TSSOP-20_4.4x6.5mm_P0.65mm, F.Cu at (205.3, 69.5)
- added Y201: Crystal, Crystal:Crystal_SMD_HC49-SD, F.Cu at (214.9, 71.9)
- moved J1 2.35 mm to (200.0, 125.1)
Connections:
- U2 pad CN10_16: Net-(U2-PadCN10_16) -> /CAN_CS
- U2 pad CN10_25: Net-(U2-PadCN10_25) -> /CAN_INTR
- U2 pad CN10_26: /enc_2_B -> /SPI2_MOSI
- U2 pad CN10_27: Net-(U2-PadCN10_27) -> /enc_2_B
- U2 pad CN10_28: /enc_2_A -> /SPI2_MISO
- U2 pad CN10_30: /recive_enable -> /SPI2_CLK
- U2 pad CN10_31: Net-(U2-PadCN10_31) -> /enc_2_A
Routing:
- net /SPI2_CLK: track 0.00 -> 70.8 mm
- net /uart_6_rx: track 61.0 -> 0.00 mm
- net /SPI2_MISO: track 0.00 -> 59.3 mm, vias 0 -> 1
- net /driver_enable: track 58.8 -> 0.00 mm, vias 1 -> 0
- net /recive_enable: track 58.8 -> 0.00 mm, vias 1 -> 0
- net /CAN_INTR: track 0.00 -> 58.5 mm, vias 0 -> 1
- net /SPI2_MOSI: track 0.00 -> 58.3 mm, vias 0 -> 1
- net /uart_6_tx: track 54.6 -> 0.00 mm, vias 1 -> 0
- net /CAN_CS: track 0.00 -> 48.2 mm
- net /Sheet607FE928/can_h: track 0.00 -> 38.5 mm
- net /Sheet607FE928/can_l: track 0.00 -> 37.8 mm
- net GND: track 13.7 -> 50.5 mm, vias 4 -> 6
- net /Sheet607FE928/can_tx: track 0.00 -> 22.7 mm, vias 0 -> 2
- net /Sheet607FE928/can_rx: track 0.00 -> 22.6 mm, vias 0 -> 2
- net Net-(C203-Pad2): track 0.00 -> 12.5 mm
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- added copper zone on B.Cu, net +5V
Other:
- board size 70.5 x 61.1 mm -> 70.5 x 76.1 mm
- board text added: "H"
- board text added: "L"

Commit message: initial
Routing:
- net /CAN_INTR: track 58.5 -> 57.2 mm
- net /SPI2_CLK: track 70.8 -> 69.5 mm
- net /SPI2_MISO: track 59.3 -> 58.0 mm
- net /SPI2_MOSI: track 58.3 -> 57.1 mm
