File: foil_controller_integrated/foil_controller_panel.kicad_pcb (KiCad board)
At the start: 2 copper layers, 100 x 152 mm, 7 parts

Commit message: initial
Routing:
- net (no net): track 0.00 -> 1.00 mm
Changed lines of the file:
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@@
     (thickness 1.6)
     (drawings 12)
-    (tracks 0)
+    (tracks 2)
     (zones 0)
     (modules 7)
@@
       (outputformat 1)
       (mirror false)
-      (drillshape 1)
+      (drillshape 0)
       (scaleselection 1)
-      (outputdirectory ""))
+      (outputdirectory "../../gerb_out/"))
   )
   (net 0 "")
@@
   (gr_line (start 95 -32) (end 95 120) (layer Edge.Cuts) (width 0.05))
   (gr_line (start -5 -32) (end 95 -32) (layer Edge.Cuts) (width 0.05))
+  (segment (start 91.5 -27) (end 91.5 -26.5) (width 0.25) (layer F.Cu) (net 0))
+  (segment (start 92 -27) (end 92 -27.5) (width 0.25) (layer B.Cu) (net 0))
 )
